File: psu.sch (KiCad schematic (older format))
At the start: 13 parts, among them P1 CONN_01X03, U5 LM7812CT, U6 LM7912CT

Commit message: did most of the layout
Parts:
- D1, D2, D3, D4: footprint Diodes_SMD:SMA_Standard -> Diodes_SMD:D_SMA
Changed lines of the file:
@@
 $Descr A4 11693 8268
 encoding utf-8
-Sheet 3 4
+Sheet 3 3
 Title ""
 Date ""
@@
 F 0 "D1" H 4150 5100 50  0000 C CNN
 F 1 "M7" H 4150 4900 50  0000 C CNN
-F 2 "Diodes_SMD:SMA_Standard" H 4150 5000 50  0001 C CNN
+F 2 "Diodes_SMD:D_SMA" H 4150 5000 50  0001 C CNN
 F 3 "" H 4150 5000 50  0000 C CNN
 	1    4150 5000
@@
 F 0 "D2" H 4200 3300 50  0000 C CNN
 F 1 "M7" H 4200 3100 50  0000 C CNN
-F 2 "Diodes_SMD:SMA_Standard" H 4200 3200 50  0001 C CNN
+F 2 "Diodes_SMD:D_SMA" H 4200 3200 50  0001 C CNN
 F 3 "" H 4200 3200 50  0000 C CNN
 	1    4200 3200
@@
 F 0 "D4" H 4200 3100 50  0000 C CNN
 F 1 "M7" H 4200 2900 50  0000 C CNN
-F 2 "Diodes_SMD:SMA_Standard" H 4200 3000 50  0001 C CNN
+F 2 "Diodes_SMD:D_SMA" H 4200 3000 50  0001 C CNN
 F 3 "" H 4200 3000 50  0000 C CNN
 	1    4200 3000
@@
 F 0 "D3" H 4150 5300 50  0000 C CNN
 F 1 "M7" H 4150 5100 50  0000 C CNN
-F 2 "Diodes_SMD:SMA_Standard" H 4150 5200 50  0001 C CNN
+F 2 "Diodes_SMD:D_SMA" H 4150 5200 50  0001 C CNN
 F 3 "" H 4150 5200 50  0000 C CNN
 	1    4150 5200
