File: amplifiers.sch (KiCad schematic (older format))
At the start: 32 parts, among them U1 LME49720, U2 LME49720, U3 LME49600, U4 LME49600

Commit message: did most of the layout
Parts:
- removed C12, C13, C16, C9: 10u, Capacitors_Tantalum_SMD:Tantalum_Case-C_EIA-6032-28_Reflow, symbol CP
- removed C14, C15: 100n, Capacitors_SMD:C_0805, symbol C
- removed R11, R12: 0R, Resistors_SMD:R_0805, symbol R
- added C12, C9: 10u, Capacitors_SMD:C_1206, symbol C
- C1, C2: footprint Capacitors_SMD:C_1206 -> Capacitors_SMD:C_0805
- C10, C11: value 100n -> 10u; footprint Capacitors_SMD:C_0805 -> Capacitors_SMD:C_1206
- U1, U2: footprint SMD_Packages:SOIC-8-N -> Housings_DIP:DIP-8_W7.62mm_Socket
Connections:
- wire segments 96 -> 85
